File: MPG.kicad_sch (KiCad schematic)
At the start: 3 parts, among them J10 DB25_Female, U14 HCPL-063A

Commit message: fix warnings
Changed lines of the file:
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@@
     (stroke (width 0) (type default) (color 0 0 0 0))
   )
-  (wire (pts (xy 132.08 83.82) (xy 132.08 85.09))
+  (wire (pts (xy 132.08 77.47) (xy 132.08 85.09))
     (stroke (width 0) (type default) (color 0 0 0 0))
   )
@@
     (stroke (width 0) (type default) (color 0 0 0 0))
   )
-  (label "IsoPWR" (at 166.37 109.22 0)
-    (effects (font (size 1.27 1.27)) (justify left bottom))
-  )
   (label "MPGB" (at 166.37 111.76 0)
     (effects (font (size 1.27 1.27)) (justify left bottom))
   )
   (label "IMPGB" (at 118.11 105.41 0)
-    (effects (font (size 1.27 1.27)) (justify left bottom))
-  )
-  (label "IsoPWR" (at 132.08 83.82 90)
-    (effects (font (size 1.27 1.27)) (justify left bottom))
-  )
-  (label "IsoPWR" (at 91.44 82.55 0)
     (effects (font (size 1.27 1.27)) (justify left bottom))
   )
@@
     (effects (font (size 1.27 1.27)) (justify left bottom))
   )
-  (hierarchical_label "IsoPower" (shape input) (at 132.08 83.82 180)
+  (hierarchical_label "IsoPower" (shape input) (at 132.08 77.47 180)
     (effects (font (size 1.27 1.27)) (justify right))
   )
@@
     (effects (font (size 1.27 1.27)) (justify right))
   )
+  (hierarchical_label "IsoPower" (shape input) (at 91.44 82.55 180)
+    (effects (font (size 1.27 1.27)) (justify right))
+  )
   (hierarchical_label "IMPGA" (shape input) (at 118.11 90.17 180)
     (effects (font (size 1.27 1.27)) (justify right))
   )
+  (hierarchical_label "IsoPower" (shape input) (at 166.37 109.22 180)
+    (effects (font (size 1.27 1.27)) (justify right))
+  )
